Commit message: Add files via upload

File: my_robot_description/urdf/my_robot.urdf.xacro (robot description, xacro)
@@ -63,45 +63,24 @@
   <!-- ## NEW: IMU Sensor Link and Joint ## -->
   <link name="imu_link">
-    <visual>
-      <geometry>
-        <box size="0.05 0.05 0.05"/>
-      </geometry>
-      <material name="black"/>
-    </visual>
-    <collision>
-      <geometry>
-        <box size="0.05 0.05 0.05"/>
-      </geometry>
-    </collision>
-    <inertial>
-      <mass value="0.01"/>
-      <inertia ixx="0.0001" ixy="0" ixz="0" iyy="0.0001" iyz="0" izz="0.0001"/>
-    </inertial>
-  </link>
-  <joint name="imu_joint" type="fixed">
-    <parent link="base_link"/> <child link="imu_link"/>
-    <origin xyz="0 0 0.15" rpy="0 0 0"/>
-  </joint>
-  <link name="gps_link">
-    <visual>
-      <geometry>
-        <box size="0.05 0.05 0.05"/>
-      </geometry>
-      <material name="black"/>
-    </visual>
-    <collision>
-      <geometry>
-        <box size="0.05 0.05 0.05"/>
-      </geometry>
-    </collision>
     <inertial>
       <mass value="0.01"/>
       <inertia ixx="1e-6" ixy="0" ixz="0" iyy="1e-6" iyz="0" izz="1e-6"/>
     </inertial>
-  </link>
-  <joint name="gps_joint" type="fixed">
+    <visual>
+      <geometry>
+        <box size="${imu_size} ${imu_size} ${imu_size}"/>
+      </geometry>
+      <material name="red"/>
+    </visual>
+    <collision>
+      <geometry>
+        <box size="${imu_size} ${imu_size} ${imu_size}"/>
+      </geometry>
+    </collision>
+  </link>
+  <joint name="imu_joint" type="fixed">
     <parent link="base_link"/>
-    <child link="gps_link"/>
-    <origin xyz="0 0 0.1" rpy="0 0 0"/>
+    <child link="imu_link"/>
+    <origin xyz="0 0 0"/>
   </joint>
   <xacro:macro name="track_housing" params="prefix side">
